File: back_panel/back_panel.sch (KiCad schematic (older format))
At the start: 5 parts, among them J1 JST-PH2, J2 JST-PH2, J3 DB9_Male_MountingHoles, J4 STEMMA JST-PH connector, U1 QT_PY

Commit message: t add pmos boaard
Parts:
- J1, J2: MPN B2B-PH-SM4-TB -> B2B-PH-SM4-TB(lf)(sn)
- J3: value DB9_Male_MountingHoles -> 191-009-113L551
- J4: MPN B4B-PH-SM4-TB -> B4B-PH-SM4-TB(lf)(sn)
Changed lines of the file:
@@
 P 3150 3350
 F 0 "J3" H 3330 3352 50  0000 L CNN
-F 1 "DB9_Male_MountingHoles" H 3330 3261 50  0000 L CNN
+F 1 "191-009-113L551" H 3330 3261 50  0000 L CNN
 F 2 "Connector_Dsub:DSUB-9_Male_Vertical_P2.77x2.84mm_MountingHoles" H 3150 3350 50  0001 C CNN
 F 3 " ~" H 3150 3350 50  0001 C CNN
@@
 F 3 "~" H 4900 4450 50  0001 C CNN
 F 4 "JST" H 0   0   50  0001 C CNN "MFR"
-F 5 "B4B-PH-SM4-TB" H 0   0   50  0001 C CNN "MPN"
+F 5 "B4B-PH-SM4-TB(lf)(sn)" H 0   0   50  0001 C CNN "MPN"
 F 6 "-" H 0   0   50  0001 C CNN "SPR"
 F 7 "-" H 0   0   50  0001 C CNN "SPN"
@@
 F 3 "~" H 1550 3550 50  0001 C CNN
 F 4 "JST" H 0   0   50  0001 C CNN "MFR"
-F 5 "B2B-PH-SM4-TB" H 0   0   50  0001 C CNN "MPN"
+F 5 "B2B-PH-SM4-TB(lf)(sn)" H 0   0   50  0001 C CNN "MPN"
 F 6 "-" H 0   0   50  0001 C CNN "SPR"
 F 7 "-" H 0   0   50  0001 C CNN "SPN"
@@
 F 3 "~" H 2150 3750 50  0001 C CNN
 F 4 "JST" H 0   0   50  0001 C CNN "MFR"
-F 5 "B2B-PH-SM4-TB" H 0   0   50  0001 C CNN "MPN"
+F 5 "B2B-PH-SM4-TB(lf)(sn)" H 0   0   50  0001 C CNN "MPN"
 F 6 "-" H 0   0   50  0001 C CNN "SPR"
 F 7 "-" H 0   0   50  0001 C CNN "SPN"
