File: front_panel/front_panel.sch (KiCad schematic (older format))
At the start: 12 parts, among them J1 Conn_Coaxial, J2 Conn_Coaxial, J3 Conn_Coaxial, J4 Conn_Coaxial, J5 Conn_Coaxial, J6 Conn_Coaxial, J7 Conn_Coaxial, J8 Conn_Coaxial

Commit message: t add pmos boaard
Parts:
- J2, J3, J4, J5, J6, J7, J8: footprint (none) -> 0my_footprints:sma_panel
Changed lines of the file:
@@
 F 0 "J2" H 2700 2675 50  0000 L CNN
 F 1 "Conn_Coaxial" H 2700 2584 50  0000 L CNN
-F 2 "" H 2600 2700 50  0001 C CNN
+F 2 "0my_footprints:sma_panel" H 2600 2700 50  0001 C CNN
 F 3 " ~" H 2600 2700 50  0001 C CNN
 	1    2600 2700
@@
 F 0 "J3" H 2700 3125 50  0000 L CNN
 F 1 "Conn_Coaxial" H 2700 3034 50  0000 L CNN
-F 2 "" H 2600 3150 50  0001 C CNN
+F 2 "0my_footprints:sma_panel" H 2600 3150 50  0001 C CNN
 F 3 " ~" H 2600 3150 50  0001 C CNN
 	1    2600 3150
@@
 F 0 "J4" H 2700 3575 50  0000 L CNN
 F 1 "Conn_Coaxial" H 2700 3484 50  0000 L CNN
-F 2 "" H 2600 3600 50  0001 C CNN
+F 2 "0my_footprints:sma_panel" H 2600 3600 50  0001 C CNN
 F 3 " ~" H 2600 3600 50  0001 C CNN
 	1    2600 3600
@@
 F 0 "J5" H 2700 4025 50  0000 L CNN
 F 1 "Conn_Coaxial" H 2700 3934 50  0000 L CNN
-F 2 "" H 2600 4050 50  0001 C CNN
+F 2 "0my_footprints:sma_panel" H 2600 4050 50  0001 C CNN
 F 3 " ~" H 2600 4050 50  0001 C CNN
 	1    2600 4050
@@
 F 0 "J6" H 2700 4475 50  0000 L CNN
 F 1 "Conn_Coaxial" H 2700 4384 50  0000 L CNN
-F 2 "" H 2600 4500 50  0001 C CNN
+F 2 "0my_footprints:sma_panel" H 2600 4500 50  0001 C CNN
 F 3 " ~" H 2600 4500 50  0001 C CNN
 	1    2600 4500
@@
 F 0 "J7" H 2700 4875 50  0000 L CNN
 F 1 "Conn_Coaxial" H 2700 4784 50  0000 L CNN
-F 2 "" H 2600 4900 50  0001 C CNN
+F 2 "0my_footprints:sma_panel" H 2600 4900 50  0001 C CNN
 F 3 " ~" H 2600 4900 50  0001 C CNN
 	1    2600 4900
@@
 F 0 "J8" H 2700 5375 50  0000 L CNN
 F 1 "Conn_Coaxial" H 2700 5284 50  0000 L CNN
-F 2 "" H 2600 5400 50  0001 C CNN
+F 2 "0my_footprints:sma_panel" H 2600 5400 50  0001 C CNN
 F 3 " ~" H 2600 5400 50  0001 C CNN
 	1    2600 5400
