File: pmos_board/coax_ch.sch (KiCad schematic (older format))
At the start: 8 parts, among them J3 Conn_Coaxial, J4 Conn_Coaxial, U2 AQY212GSZ

Commit message: Update to pmosboard
Changed lines of the file:
@@
 $Descr A4 11693 8268
 encoding utf-8
-Sheet 2 9
+Sheet 2 17
 Title ""
 Date ""
@@
 AR Path="/5FF8BA79/5FF2E16D" Ref="J16"  Part="1"
 AR Path="/5FF8BA7C/5FF2E16D" Ref="J18"  Part="1"
-F 0 "J4" H 7328 4688 50  0000 C CNN
+F 0 "J18" H 7328 4688 50  0000 C CNN
 F 1 "Conn_Coaxial" H 7328 4597 50  0000 C CNN
 F 2 "Connector_Coaxial:SMA_Amphenol_132134_Vertical" H 7400 4450 50  0001 C CNN
@@
 AR Path="/5FF8BA79/5FF2F135" Ref="J15"  Part="1"
 AR Path="/5FF8BA7C/5FF2F135" Ref="J17"  Part="1"
-F 0 "J3" H 7228 3738 50  0000 C CNN
+F 0 "J17" H 7228 3738 50  0000 C CNN
 F 1 "Conn_Coaxial" H 7228 3647 50  0000 C CNN
 F 2 "Connector_Coaxial:SMA_Amphenol_132134_Vertical" H 7300 3500 50  0001 C CNN
@@
 AR Path="/5FF8BA79/5FF33823" Ref="#PWR049"  Part="1"
 AR Path="/5FF8BA7C/5FF33823" Ref="#PWR055"  Part="1"
-F 0 "#PWR013" H 7300 3450 50  0001 C CNN
+F 0 "#PWR055" H 7300 3450 50  0001 C CNN
 F 1 "GND" H 7305 3527 50  0000 C CNN
 F 2 "" H 7300 3700 50  0001 C CNN
@@
 AR Path="/5FF8BA79/5FF33D5E" Ref="#PWR048"  Part="1"
 AR Path="/5FF8BA7C/5FF33D5E" Ref="#PWR054"  Part="1"
-F 0 "#PWR012" H 7400 4400 50  0001 C CNN
+F 0 "#PWR054" H 7400 4400 50  0001 C CNN
 F 1 "GND" H 7405 4477 50  0000 C CNN
 F 2 "" H 7400 4650 50  0001 C CNN
@@
 AR Path="/5FF8BA79/6031686D" Ref="U8"  Part="1"
 AR Path="/5FF8BA7C/6031686D" Ref="U9"  Part="1"
-F 0 "U2" H 6200 3925 50  0000 C CNN
+F 0 "U9" H 6200 3925 50  0000 C CNN
 F 1 "AQY212GSZ" H 6200 3834 50  0000 C CNN
 F 2 "0my_footprints:AQY211G2S_samacsys" H 6000 3400 50  0001 L CIN
@@
 AR Path="/5FF8BA79/6031A62E" Ref="R15"  Part="1"
 AR Path="/5FF8BA7C/6031A62E" Ref="R16"  Part="1"
-F 0 "R9" V 5545 3050 50  0000 C CNN
+F 0 "R16" V 5545 3050 50  0000 C CNN
 F 1 "390" V 5636 3050 50  0000 C CNN
 F 2 "Resistor_SMD:R_0603_1608Metric_Pad1.05x0.95mm_HandSolder" V 5790 3040 50  0001 C CNN
@@
 AR Path="/5FF8BA79/60321698" Ref="#PWR0121"  Part="1"
 AR Path="/5FF8BA7C/60321698" Ref="#PWR0123"  Part="1"
-F 0 "#PWR0108" H 5900 3750 50  0001 C CNN
+F 0 "#PWR0123" H 5900 3750 50  0001 C CNN
 F 1 "GNDD" H 5904 3845 50  0000 C CNN
 F 2 "" H 5900 4000 50  0001 C CNN
@@
 AR Path="/5FF8BA79/6033C70A" Ref="C14"  Part="1"
 AR Path="/5FF8BA7C/6033C70A" Ref="C16"  Part="1"
-F 0 "C2" H 6465 4646 50  0000 L CNN
+F 0 "C16" H 6465 4646 50  0000 L CNN
 F 1 "100uF" H 6465 4555 50  0000 L CNN
 F 2 "Capacitor_SMD:C_1206_3216Metric_Pad1.42x1.75mm_HandSolder" H 6388 4450 50  0001 C CNN
@@
 AR Path="/5FF8BA79/6033D81C" Ref="#PWR0127"  Part="1"
 AR Path="/5FF8BA7C/6033D81C" Ref="#PWR0129"  Part="1"
-F 0 "#PWR0102" H 6900 4550 50  0001 C CNN
+F 0 "#PWR0129" H 6900 4550 50  0001 C CNN
 F 1 "GND" H 6905 4627 50  0000 C CNN
 F 2 "" H 6900 4800 50  0001 C CNN
@@
 AR Path="/5FF8BA79/6033DC0A" Ref="#PWR0128"  Part="1"
 AR Path="/5FF8BA7C/6033DC0A" Ref="#PWR0130"  Part="1"
-F 0 "#PWR0103" H 6350 4500 50  0001 C CNN
+F 0 "#PWR0130" H 6350 4500 50  0001 C CNN
 F 1 "GND" H 6355 4577 50  0000 C CNN
 F 2 "" H 6350 4750 50  0001 C CNN
@@
 AR Path="/5FF8BA79/6033F02D" Ref="R7"  Part="1"
 AR Path="/5FF8BA7C/6033F02D" Ref="R8"  Part="1"
-F 0 "R1" H 7068 3696 50  0000 L CNN
+F 0 "R8" H 7068 3696 50  0000 L CNN
 F 1 "10K 0.1%" H 7068 3605 50  0000 L CNN
 F 2 "Resistor_SMD:R_0603_1608Metric_Pad1.05x0.95mm_HandSolder" V 7040 3640 50  0001 C CNN
@@
 AR Path="/5FF8BA79/6033F7F5" Ref="#PWR0137"  Part="1"
 AR Path="/5FF8BA7C/6033F7F5" Ref="#PWR0138"  Part="1"
-F 0 "#PWR0131" H 7000 3550 50  0001 C CNN
+F 0 "#PWR0138" H 7000 3550 50  0001 C CNN
 F 1 "GND" H 7005 3627 50  0000 C CNN
 F 2 "" H 7000 3800 50  0001 C CNN
@@
 AR Path="/5FF8BA79/60340756" Ref="C15"  Part="1"
 AR Path="/5FF8BA7C/60340756" Ref="C17"  Part="1"
-F 0 "C3" H 7015 4696 50  0000 L CNN
+F 0 "C17" H 7015 4696 50  0000 L CNN
 F 1 "100uF" H 7015 4605 50  0000 L CNN
 F 2 "Capacitor_SMD:C_1206_3216Metric_Pad1.42x1.75mm_HandSolder" H 6938 4500 50  0001 C CNN
@@
 AR Path="/5FF8BA79/6033B87E" Ref="FB7"  Part="1"
 AR Path="/5FF8BA7C/6033B87E" Ref="FB8"  Part="1"
-F 0 "FB1" V 6376 4450 50  0000 C CNN
+F 0 "FB8" V 6376 4450 50  0000 C CNN
 F 1 "Ferrite_Bead" V 6467 4450 50  0000 C CNN
 F 2 "Inductor_SMD:L_0805_2012Metric_Pad1.15x1.40mm_HandSolder" V 6580 4450 50  0001 C CNN
@@
 Wire Wire Line
 	6900 4450 7200 4450
+$Sheet
+S 7950 1650 1100 450
+U 600A1E9E
+F0 "Sheet600A1E9D" 50
+F1 "temp.sch" 50
+$EndSheet
 $EndSCHEMATC
