File: pmos_board/pmos_board.kicad_pcb (KiCad board)
At the start: 2 copper layers, 30 x 100 mm, 70 parts, among them J1 Conn_01x04, J10 Conn_Coaxial, J11 Conn_Coaxial, J12 Conn_Coaxial, J13 Conn_Coaxial, J14 Conn_Coaxial, J15 Conn_Coaxial, J16 Conn_Coaxial, J17 Conn_Coaxial, J18 Conn_Coaxial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

Commit message: Update to pmosboard
Connections:
- J1 pad 1: /scl -> GNDD
- J1 pad 2: /sda -> +3V3
- J1 pad 3: +3V3 -> /sda
- J1 pad 4: GNDD -> /scl
Routing:
- net +3V3: track 22.0 -> 34.5 mm
- net GNDD: track 146.9 -> 140.7 mm, vias 13 -> 12
- net /sda: track 18.1 -> 14.4 mm
- net /scl: track 18.3 -> 15.3 mm
