File: pmos_board/pmos_board.sch (KiCad schematic (older format))
At the start: 6 parts, among them J1 Conn_01x04, U1 TCA9534APWR

Commit message: Update to pmosboard
Parts:
- J1: symbol 0my_intf:Conn_01x04_i2c -> 0my_intf:JST_SH_Conn_01x04_i2c
Changed lines of the file:
@@
 $Descr A4 11693 8268
 encoding utf-8
-Sheet 1 9
+Sheet 1 17
 Title ""
 Date ""
@@
 $EndComp
 $Comp
-L 0my_intf:Conn_01x04_i2c J1
+L 0my_intf:JST_SH_Conn_01x04_i2c J1
 U 1 1 5FF52F8D
 P 4350 2950
