File: back_v3/back_v3.kicad_pcb (KiCad board)
At the start: 2 copper layers, 103 x 30.5 mm, 12 parts, among them J1 JST-PH2, J2 JST-PH2, J3 191-009-113L551, J4 STEMMA JST-PH connector, J5 JST-SH, U1 QT_PY

Commit message: update back_v3
Parts:
- added R5: 3.3K, Resistor_SMD:R_0603_1608Metric_Pad1.05x0.95mm_HandSolder, F.Cu at (143.0, 122.0)
- added U2: AQY212, Package_SO:SO-4_4.4x4.3mm_P2.54mm, F.Cu at (136.0, 121.0)
- J2: value JST-PH2 -> JST-SH; footprint Connector_JST:JST_PH_B2B-PH-SM4-TB_1x02-1MP_P2.00mm_Vertical -> Connector_JST:JST_SH_BM04B-SRSS-TB_1x04-1MP_P1.00mm_Vertical
- moved J2 15.2 mm to (124.0, 121.0)
- moved H1 7.72 mm to (109.6, 111.3)
- moved J5 0.20 mm to (124.0, 102.0), turned to 0 degrees
Connections:
- net Net-(D1-Pad2) renamed +5V
- J2 pad 1: Net-(J2-Pad1) -> /GND_I2C
- J5 pad 1: /SCL -> /GND_I2C
- J5 pad 2: /SDA -> /3V_I2C
- J5 pad 3: /3V_I2C -> /SDA
- J5 pad 4: /GND_I2C -> /SCL
- U1 pad 2: Net-(J2-Pad1) -> Net-(U1-Pad2)
- U1 pad 3: Net-(J2-Pad2) -> Net-(U1-Pad3)
Routing:
- net /3V_I2C: track 94.3 -> 134.4 mm
- net /GND_I2C: track 91.2 -> 130.9 mm, vias 0 -> 2
- net Net-(J2-Pad1): track 38.7 -> 0.00 mm
- net +5V: track 22.3 -> 54.3 mm
- net /SDA: track 67.4 -> 89.3 mm
- net /SCL: track 54.5 -> 76.4 mm
- net Net-(J2-Pad2): track 30.0 -> 15.1 mm
- net Net-(R5-Pad2): track 0.00 -> 3.24 mm
