File: back_v3/back_v3.sch (KiCad schematic (older format))
At the start: 12 parts, among them J1 JST-PH2, J2 JST-PH2, J3 191-009-113L551, J4 STEMMA JST-PH connector, J5 JST-SH, U1 QT_PY

Commit message: update back_v3
Parts:
- removed J2: JST-PH2, Connector_JST:JST_PH_B2B-PH-SM4-TB_1x02-1MP_P2.00mm_Vertical, symbol Connector:Conn_01x02_Female
- added J2: JST-SH, Connector_JST:JST_SH_BM04B-SRSS-TB_1x04-1MP_P1.00mm_Vertical, symbol 0my_intf:JST_SH_Conn_01x04_i2c
- added R5: 2K, Resistor_SMD:R_0603_1608Metric_Pad1.05x0.95mm_HandSolder, symbol Device:R_US
- added U2: AQY212, Package_SO:SO-4_4.4x4.3mm_P2.54mm, symbol Relay_SolidState:ASSR-1218
- D1: LCSC (none) -> C117485; MPN (none) -> BAT60AE6327
- H1: footprint MountingHole:MountingHole_8.4mm_M8 -> 0my_footprints:MountingHole_8.4mm_PJ-066
- J5: symbol 0my_intf:Conn_01x04_i2c -> 0my_intf:JST_SH_Conn_01x04_i2c
- R1: value R_Small_US -> 10K; LCAC (none) -> C25804; MPN (none) -> 0603WAF1002T5E
- R2: value R_Small_US -> 10K; LCSC (none) -> C25804; MPN (none) -> 0603WAF1002T5E
- R3: LCSC (none) -> C22975; MPN (none) -> 0603WAF2001T5E
- R4: LCSC (none) -> C22978; MPN (none) -> 0603WAF3301T5E
Connections:
- net labels added: +5V
- wire segments 16 -> 17
- no-connect marks 4 -> 6
Changed lines of the file:
@@
-$EndComp
-$Comp
-L Connector:Conn_01x02_Female J2
-U 1 1 5FCB4462
-P 6700 4200
-F 0 "J2" H 6800 4150 50  0000 C CNN
-F 1 "JST-PH2" H 6600 4300 50  0000 C CNN
-F 2 "Connector_JST:JST_PH_B2B-PH-SM4-TB_1x02-1MP_P2.00mm_Vertical" H 6700 4200 50  0001 C CNN
-F 3 "~" H 6700 4200 50  0001 C CNN
-F 4 "JST" H 4550 450 50  0001 C CNN "MFR"
-F 5 "B2B-PH-SM4-TB(lf)(sn)" H 4550 450 50  0001 C CNN "MPN"
-F 6 "-" H 4550 450 50  0001 C CNN "SPR"
-F 7 "-" H 4550 450 50  0001 C CNN "SPN"
-F 8 "-" H 4550 450 50  0001 C CNN "SPURL"
-	1    6700 4200
-	-1   0    0    -1
 $EndComp
 $Comp
@@
 NoConn ~ 7850 4400
 $Comp
-L 0my_intf:Conn_01x04_i2c J5
+L 0my_intf:JST_SH_Conn_01x04_i2c J5
 U 1 1 5FFC6E13
 P 6050 4450
@@
 P 5950 3550
 F 0 "R1" V 5745 3550 50  0000 C CNN
-F 1 "R_Small_US" V 5836 3550 50  0000 C CNN
+F 1 "10K" V 5836 3550 50  0000 C CNN
 F 2 "Resistor_SMD:R_0603_1608Metric_Pad1.05x0.95mm_HandSolder" H 5950 3550 50  0001 C CNN
 F 3 "~" H 5950 3550 50  0001 C CNN
+F 4 "C25804" V 5950 3550 50  0001 C CNN "LCAC"
+F 5 "0603WAF1002T5E" V 5950 3550 50  0001 C CNN "MPN"
 	1    5950 3550
 	0    1    1    0
@@
 P 5950 3850
 F 0 "R2" V 5745 3850 50  0000 C CNN
-F 1 "R_Small_US" V 5836 3850 50  0000 C CNN
+F 1 "10K" V 5836 3850 50  0000 C CNN
 F 2 "Resistor_SMD:R_0603_1608Metric_Pad1.05x0.95mm_HandSolder" H 5950 3850 50  0001 C CNN
 F 3 "~" H 5950 3850 50  0001 C CNN
+F 4 "0603WAF1002T5E" V 5950 3850 50  0001 C CNN "MPN"
+F 5 "C25804" V 5950 3850 50  0001 C CNN "LCSC"
 	1    5950 3850
 	0    1    1    0
@@
 F 2 "Diode_SMD:D_SOD-323" H 7750 3025 50  0001 C CNN
 F 3 "https://www.infineon.com/dgdl/Infineon-BAT60ASERIES-DS-v01_01-en.pdf?fileId=db3a304313d846880113def70c9304a9" H 7750 3200 50  0001 C CNN
+F 4 "C117485" H 7750 3200 50  0001 C CNN "LCSC"
+F 5 "BAT60AE6327" H 7750 3200 50  0001 C CNN "MPN"
 	1    7750 3200
 	-1   0    0    1
@@
 F 2 "Resistor_SMD:R_0603_1608Metric_Pad1.05x0.95mm_HandSolder" V 7540 3340 50  0001 C CNN
 F 3 "~" H 7500 3350 50  0001 C CNN
+F 4 "C22975" H 7500 3350 50  0001 C CNN "LCSC"
+F 5 "0603WAF2001T5E" H 7500 3350 50  0001 C CNN "MPN"
 	1    7500 3350
 	1    0    0    -1
@@
 F 2 "Resistor_SMD:R_0603_1608Metric_Pad1.05x0.95mm_HandSolder" V 7690 3490 50  0001 C CNN
 F 3 "~" H 7650 3500 50  0001 C CNN
+F 4 "C22978" V 7650 3500 50  0001 C CNN "LCSC"
+F 5 "0603WAF3301T5E" V 7650 3500 50  0001 C CNN "MPN"
 	1    7650 3500
 	0    -1   1    0
@@
 F 0 "H1" H 8650 2196 50  0000 L CNN
 F 1 "MountingHole" H 8650 2105 50  0000 L CNN
-F 2 "MountingHole:MountingHole_8.4mm_M8" H 8550 2150 50  0001 C CNN
+F 2 "0my_footprints:MountingHole_8.4mm_PJ-066" H 8550 2150 50  0001 C CNN
 F 3 "~" H 8550 2150 50  0001 C CNN
 	1    8550 2150
 	1    0    0    -1
 $EndComp
+NoConn ~ 6900 4200
+NoConn ~ 6900 4300
+$Comp
+L 0my_intf:JST_SH_Conn_01x04_i2c J2
+U 1 1 601BF973
+P 6050 5450
+F 0 "J2" H 6260 5450 50  0000 L CNN
+F 1 "JST-SH" H 6260 5359 50  0000 L CNN
+F 2 "Connector_JST:JST_SH_BM04B-SRSS-TB_1x04-1MP_P1.00mm_Vertical" H 6050 5450 50  0001 C CNN
+F 3 "~" H 6050 5450 50  0001 C CNN
+F 4 "JST-SH-BM04B-SRSS-TB" H 6050 5450 50  0001 C CNN "MPN"
+	1    6050 5450
+	1    0    0    -1
+$EndComp
+Text Label 5850 5550 2    50   ~ 0
+SDA
+Text Label 5850 5650 2    50   ~ 0
+SCL
+Text Label 5850 5350 2    50   ~ 0
+GND_I2C
+$Comp
+L Relay_SolidState:ASSR-1218 U2
+U 1 1 601C7996
+P 5250 5750
+F 0 "U2" V 5296 5570 50  0000 R CNN
+F 1 "AQY212" V 5205 5570 50  0000 R CNN
+F 2 "Package_SO:SO-4_4.4x4.3mm_P2.54mm" H 5050 5550 50  0001 L CIN
+F 3 "https://docs.broadcom.com/docs/AV02-0173EN" H 5250 5750 50  0001 L CNN
+F 4 "C129283" H 5250 5750 50  0001 C CNN "LCSC"
+F 5 "AQY212GSZ" V 5250 5750 50  0001 C CNN "MPN"
+	1    5250 5750
+	0    -1   -1   0
+$EndComp
+Wire Wire Line
+	5850 5450 5350 5450
+Text Label 5150 5450 2    50   ~ 0
+3V_I2C
+Text Label 5350 6050 0    50   ~ 0
+GND_I2C
+$Comp
+L Device:R_US R5
+U 1 1 601CADF5
+P 5000 6050
+F 0 "R5" V 5100 5850 50  0000 C CNN
+F 1 "2K" V 5100 6050 50  0000 C CNN
+F 2 "Resistor_SMD:R_0603_1608Metric_Pad1.05x0.95mm_HandSolder" V 5040 6040 50  0001 C CNN
+F 3 "~" H 5000 6050 50  0001 C CNN
+F 4 "C22975" V 5000 6050 50  0001 C CNN "LCSC"
+F 5 "0603WAF2001T5E" V 5000 6050 50  0001 C CNN "MPN"
+	1    5000 6050
+	0    -1   1    0
+$EndComp
+$Comp
+L power:+5V #PWR0102
+U 1 1 601CC20D
+P 7500 3200
+F 0 "#PWR0102" H 7500 3050 50  0001 C CNN
+F 1 "+5V" H 7515 3373 50  0000 C CNN
+F 2 "" H 7500 3200 50  0001 C CNN
+F 3 "" H 7500 3200 50  0001 C CNN
+	1    7500 3200
+	1    0    0    -1
+$EndComp
+$Comp
+L power:+5V #PWR0103
+U 1 1 601CCA0F
+P 4850 6050
+F 0 "#PWR0103" H 4850 5900 50  0001 C CNN
+F 1 "+5V" V 4865 6178 50  0000 L CNN
+F 2 "" H 4850 6050 50  0001 C CNN
+F 3 "" H 4850 6050 50  0001 C CNN
+	1    4850 6050
+	0    -1   -1   0
+$EndComp
 $EndSCHEMATC
